File: matrix.sch (KiCad schematic (older format))
At the start: 72 parts, among them K1 SHIFT, K10 O, K11 P, K12 BKSP, K13 CTRL, K14 A, K15 S, K16 D, K17 F, K18 G, K19 H, K2 Q, K20 J, K21 K, K22 L, K23 UP, K24 ENTER, K25 FN, K26 Z, K27 X, K28 C, K29 V, K3 W, K30 SPACE, K31 B, K32 N, K33 M, K34 LEFT, K35 DOWN, K36 RIGHT, K4 E, K5 R, K6 T, K7 Y, K8 U, K9 I

Commit message: Enrutado
Connections:
- net row0 is gone; now on net col11: D1.1 (K), D10.1 (K), D11.1 (K), D12.1 (K), D2.1 (K), D3.1 (K), D4.1 (K), D5.1 (K), D6.1 (K), D7.1 (K), D8.1 (K), D9.1 (K)
- net row1 is gone; now on net col11: D13.1 (K), D14.1 (K), D15.1 (K), D16.1 (K), D17.1 (K), D18.1 (K), D19.1 (K), D20.1 (K), D21.1 (K), D22.1 (K), D23.1 (K), D24.1 (K)
Changed lines of the file:
@@
 	0    -1   -1   0
 $EndComp
+Wire Wire Line
+	1225 4775 1975 4775
 $Comp
 L keyboard_parts:KEYSW K26
@@
 	0    -1   -1   0
 $EndComp
+Connection ~ 1975 4775
+Wire Wire Line
+	1975 4775 2725 4775
 $Comp
 L keyboard_parts:KEYSW K27
@@
 	0    -1   -1   0
 $EndComp
+Connection ~ 3475 4775
+Wire Wire Line
+	3475 4775 4225 4775
+Connection ~ 2725 4775
+Wire Wire Line
+	2725 4775 3475 4775
 $Comp
 L keyboard_parts:KEYSW K29
@@
 	0    -1   -1   0
 $EndComp
+Connection ~ 4975 4775
+Wire Wire Line
+	4975 4775 5725 4775
 $Comp
 L keyboard_parts:KEYSW K31
@@
 	0    -1   -1   0
 $EndComp
+Connection ~ 6475 4775
+Connection ~ 5725 4775
+Wire Wire Line
+	5725 4775 6475 4775
+Connection ~ 4225 4775
+Wire Wire Line
+	4225 4775 4975 4775
+Wire Wire Line
+	6475 4775 7225 4775
 $Comp
 L Device:D D33
@@
 	1    0    0    -1
 $EndComp
+Connection ~ 7225 4775
+Wire Wire Line
+	7225 4775 7975 4775
 $Comp
 L keyboard_parts:KEYSW K34
@@
 	0    -1   -1   0
 $EndComp
+Connection ~ 7975 4775
+Wire Wire Line
+	7975 4775 8725 4775
 $Comp
 L keyboard_parts:KEYSW K35
@@
 	0    -1   -1   0
 $EndComp
+Connection ~ 8725 4775
 $Comp
 L keyboard_parts:KEYSW K36
@@
 Wire Wire Line
 	9325 3625 9325 4475
+Wire Wire Line
+	10075 3625 10075 3925
 Text GLabel 1000 3075 0    50   Input ~ 0
 row0
 Wire Wire Line
+	8725 4775 9475 4775
+Wire Wire Line
 	1225 3925 1000 3925
 Connection ~ 1225 3925
+Wire Wire Line
+	1225 4775 1000 4775
+Connection ~ 1225 4775
 Text GLabel 1000 3925 0    50   Input ~ 0
 row1
@@
 Wire Wire Line
 	9325 2775 9325 3625
+Wire Wire Line
+	10075 2775 10075 3075
 Wire Wire Line
 	1000 3075 1225 3075
@@
 col11
 Wire Wire Line
-	9475 4775 8725 4775
-Connection ~ 1225 4775
-Wire Wire Line
-	1225 4775 1000 4775
-Connection ~ 1975 4775
-Wire Wire Line
-	1975 4775 1225 4775
-Connection ~ 2725 4775
-Wire Wire Line
-	2725 4775 1975 4775
-Connection ~ 3475 4775
-Wire Wire Line
-	3475 4775 2725 4775
-Connection ~ 4225 4775
-Wire Wire Line
-	4225 4775 3475 4775
-Connection ~ 4975 4775
-Wire Wire Line
-	4975 4775 4225 4775
-Connection ~ 5725 4775
-Wire Wire Line
-	5725 4775 4975 4775
-Connection ~ 6475 4775
-Wire Wire Line
-	6475 4775 5725 4775
-Connection ~ 7225 4775
-Wire Wire Line
-	7225 4775 6475 4775
-Connection ~ 7975 4775
-Wire Wire Line
-	7975 4775 7225 4775
-Connection ~ 8725 4775
-Wire Wire Line
-	8725 4775 7975 4775
-Wire Wire Line
-	10075 3625 10075 4475
-Wire Wire Line
-	10075 2775 10075 3625
+	9475 3075 10075 3075
+Connection ~ 9475 3075
+Connection ~ 10075 3075
+Wire Wire Line
+	10075 3075 10075 3625
+Wire Wire Line
+	9475 3925 10075 3925
+Connection ~ 9475 3925
+Connection ~ 10075 3925
+Wire Wire Line
+	10075 3925 10075 4475
 $EndSCHEMATC
